File: pure.kicad_sch (KiCad schematic)
At the start: 2 parts, among them J1 TX, J6 RX

Commit message: add whole module PCB
Connections:
- net RELAY_POWER: now reaches J6.7 (Pin_7)
Changed lines of the file:
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@@
 	(wire
 		(pts
-			(xy 171.45 33.02) (xy 151.13 33.02)
+			(xy 177.8 33.02) (xy 151.13 33.02)
 		)
 		(stroke
@@
 	(wire
 		(pts
-			(xy 151.13 38.1) (xy 171.45 38.1)
+			(xy 151.13 38.1) (xy 177.8 38.1)
 		)
 		(stroke
@@
 	(wire
 		(pts
-			(xy 151.13 43.18) (xy 171.45 43.18)
+			(xy 151.13 43.18) (xy 177.8 43.18)
 		)
 		(stroke
@@
 	(wire
 		(pts
-			(xy 151.13 27.94) (xy 171.45 27.94)
+			(xy 151.13 27.94) (xy 177.8 27.94)
 		)
 		(stroke
@@
 	(global_label "I_LINE_IN"
 		(shape input)
-		(at 171.45 43.18 0)
+		(at 177.8 43.18 0)
 		(fields_autoplaced yes)
 		(effects
@@
 		)
 		(property "Intersheetrefs" "${INTERSHEET_REFS}"
-			(at 184.5519 43.18 0)
+			(at 190.9019 43.18 0)
 			(effects
 				(font
@@
 	(global_label "RX0"
 		(shape output)
-		(at 171.45 27.94 0)
+		(at 177.8 27.94 0)
 		(fields_autoplaced yes)
 		(effects
@@
 		)
 		(property "Intersheetrefs" "${INTERSHEET_REFS}"
-			(at 178.6736 27.94 0)
+			(at 185.0236 27.94 0)
 			(effects
 				(font
@@
 		)
 	)
+	(global_label "RELAY_POWER"
+		(shape output)
+		(at 156.21 40.64 0)
+		(fields_autoplaced yes)
+		(effects
+			(font
+				(size 1.524 1.524)
+			)
+			(justify left)
+		)
+		(property "Intersheetrefs" "${INTERSHEET_REFS}"
+			(at 174.6823 40.64 0)
+			(effects
+				(font
+					(size 1.27 1.27)
+				)
+				(justify left)
+				(hide yes)
+			)
+		)
+	)
 	(global_label "Q_LINE_IN"
 		(shape input)
@@
 	(global_label "RX180"
 		(shape output)
-		(at 171.45 33.02 0)
+		(at 177.8 33.02 0)
 		(fields_autoplaced yes)
 		(effects
@@
 		)
 		(property "Intersheetrefs" "${INTERSHEET_REFS}"
-			(at 181.5764 33.02 0)
+			(at 187.9264 33.02 0)
 			(effects
 				(font
@@
 	(symbol
 		(lib_id "power:+10V")
-		(at 171.45 38.1 270)
+		(at 177.8 38.1 270)
 		(unit 1)
 		(exclude_from_sim no)
@@
 		(fields_autoplaced yes)
 		(property "Reference" "#PWR08"
-			(at 167.64 38.1 0)
+			(at 173.99 38.1 0)
 			(effects
 				(font
@@
 		)
 		(property "Value" "+10V"
-			(at 175.26 38.0999 90)
+			(at 181.61 38.0999 90)
 			(effects
 				(font
@@
 		)
 		(property "Footprint" ""
-			(at 171.45 38.1 0)
+			(at 177.8 38.1 0)
 			(effects
 				(font
@@
 		)
 		(property "Datasheet" ""
-			(at 171.45 38.1 0)
+			(at 177.8 38.1 0)
 			(effects
 				(font
@@
 		)
 		(property "Description" "Power symbol creates a global label with name \"+10V\""
-			(at 171.45 38.1 0)
-			(effects
-				(font
+			(at 177.8 38.1 0)
+			(effects
+				(font
